File: 遥控器/遥控器.kicad_pcb (KiCad board)
At the start: 2 copper layers, 150 x 90.8 mm, 61 parts, among them J1 Conn_01x01_Pin, J2 Conn_01x01_Pin, J3 USB_C_Receptacle_USB2.0, SW1 SK12F14G5, SW10 SW_Push, SW11 SW_Push, SW12 SW_Push, SW13 SW_Push, SW14 SW_Push, SW2 SW_Push, SW3 SW_Push, SW4 SW_Push, SW5 SW_Push, SW6 SW_Push, SW7 SW_Push, SW8 SW_Push, SW9 SW_Push, U1 SX1308, U2 IPS_1.14_135X240_ST7789_13P顶层, U3 STM32F103RCTx, U4 ME6206A33M3G, U5 2.4G-UART, U6 W25Q128JVS, U8 10k, U9 10k, Y1 8M

Commit message: 完成pcb绘制
Parts:
- added J3: Conn_01x01_Pin, Connector_Wire:SolderWirePad_1x01_SMD_1x2mm, F.Cu at (127.5, 125.7)
- added J4: Conn_01x01_Pin, Connector_Wire:SolderWirePad_1x01_SMD_1x2mm, F.Cu at (125.3, 125.7)
- added J5: Conn_01x01_Pin, Connector_Wire:SolderWirePad_1x01_SMD_1x2mm, F.Cu at (123.3, 125.7)
- added J6: Conn_01x01_Pin, Connector_Wire:SolderWirePad_1x01_SMD_1x2mm, F.Cu at (121.2, 125.7)
- BAT+: renamed from J1; moved to B.Cu
- BAT-: renamed from J2; moved to B.Cu
- C1, C10, C19, C2, C3, C4, C9, L2, R2, R6, R8: moved to B.Cu
- moved U1 125.0 mm to (163.6, 116.7)
- moved D1 116.9 mm to (163.7, 113.3)
- moved L1 116.7 mm to (168.7, 115.0), turned to -90 degrees
- moved U4 112.0 mm to (152.2, 114.2), turned to 90 degrees
- moved C6 101.9 mm to (167.2, 119.7)
- moved C5 101.6 mm to (163.9, 119.7), turned to 180 degrees
- moved Y1 101.2 mm to (164.8, 100.2), turned to -90 degrees
- moved C12 96.0 mm to (160.2, 113.7), turned to -90 degrees
- moved U6 94.1 mm to (130.9, 96.2)
- moved C13 92.9 mm to (158.5, 113.7), turned to -90 degrees
- moved R1 92.1 mm to (160.2, 116.9), turned to -90 degrees
- moved C14 91.4 mm to (155.1, 116.9), turned to -90 degrees
- moved C15 90.4 mm to (156.8, 116.9), turned to -90 degrees
- moved C7 88.6 mm to (156.8, 113.7), turned to -90 degrees
- moved R3 87.1 mm to (158.5, 116.9), turned to 90 degrees
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- renumbered J3 to J7
Connections:
- net Net-(D1-A) renamed /SW
- J7 pad S1: unconnected-(J3-SHIELD-PadS1) -> GND
- U2 pad 4: /SPI2_SCL -> /SPI1_SCL
- U3 pad 29: unconnected-(U3-PB10-Pad29) -> /S12
- U3 pad 30: unconnected-(U3-PB11-Pad30) -> /S11
- U3 pad 45: unconnected-(U3-PA12-Pad45) -> /S1
- U3 pad 46: unconnected-(U3-PA13-Pad46) -> /SWDIO
- U3 pad 49: unconnected-(U3-PA14-Pad49) -> /SWCLK
- U3 pad 50: /S1 -> /S2
- U3 pad 51: /S2 -> /S4
- U3 pad 53: /S4 -> unconnected-(U3-PC12-Pad53)
- U3 pad 54: /S5 -> /S10
- U3 pad 55: /S6 -> /S7
- U3 pad 56: /S7 -> /S6
- U3 pad 58: /S9 -> /S5
- U3 pad 59: /S10 -> /S9
- U3 pad 61: /S11 -> unconnected-(U3-PB8-Pad61)
- U3 pad 62: /S12 -> unconnected-(U3-PB9-Pad62)
Routing:
- net +3.3V: track 0.00 -> 311.7 mm, vias 0 -> 10
- net /S8: track 0.00 -> 59.1 mm
- net /AD1: track 0.00 -> 58.5 mm, vias 0 -> 1
- net /S2: track 0.00 -> 56.9 mm, vias 0 -> 2
- net /S4: track 0.00 -> 55.8 mm, vias 0 -> 2
- net /S6: track 0.00 -> 53.7 mm
- net +BATT: track 0.00 -> 52.0 mm, vias 0 -> 1
- net /S9: track 0.00 -> 52.0 mm, vias 0 -> 2
- net /S5: track 0.00 -> 50.8 mm
- net /S10: track 0.00 -> 49.7 mm, vias 0 -> 4
- net /S11: track 0.00 -> 46.6 mm
- net /AD3: track 0.00 -> 45.8 mm, vias 0 -> 1
- net /S1: track 0.00 -> 44.0 mm, vias 0 -> 2
- net /SWCLK: track 0.00 -> 40.9 mm, vias 0 -> 2
- net /SWDIO: track 0.00 -> 40.7 mm, vias 0 -> 2
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- added copper zone on F.Cu, net +3.3V
- added copper zone on F.Cu, net +5V
- added copper zone on F.Cu, net +BATT
- added copper zone on F.Cu, net /SW
- added copper zone on B.Cu, net GND
- added copper zone on F.Cu, net GND
- added copper zone on In2.Cu, net GND
Other:
- copper layers 2 -> 4
- board text added: "3V3"
- board text added: "A"
- board text added: "B"
- board text added: "CLK"
- board text added: "DIO"
- board text added: "GND"
- board text added: "JLCJLCJLCJLC"
- board text added: "L1"
- board text added: "L2"
- board text added: "OFF"
- board text added: "ON"
- board text added: "X"
- board text added: "Y"
- board text added: "https://github.com/CodonNine"

Commit message: 飞控原理图完成
Parts:
- added C5: 0.1u, Capacitor_SMD:C_0603_1608Metric, F.Cu at (157.2, 93.0)
- added G***: LOGO, Symbol:simpleflight_copper, F.Cu at (148.0, 69.4)
- added G***: LOGO, Symbol:simpleflight, B.Cu at (148.0, 95.0)
- added REF**: OSHW-Logo_11.4x12mm_SilkScreen, Symbol:OSHW-Logo_11.4x12mm_SilkScreen, B.Cu at (98.8, 104.0)
- added REF**: KiCad-Logo2_8mm_SilkScreen, Symbol:KiCad-Logo2_8mm_SilkScreen, B.Cu at (97.6, 116.6)
- C1, C2, C3, C4, L2, R6, R8: moved to F.Cu
- C10: renamed from C9; moved to F.Cu
- C11: renamed from C10; moved to F.Cu
- moved R4 13.9 mm to (161.8, 107.5), turned to 90 degrees
- moved R7 12.8 mm to (160.2, 107.5), turned to -90 degrees
- moved R6 10.7 mm to (158.5, 107.5), turned to -90 degrees
- moved C4 10.5 mm to (156.8, 107.5), turned to -90 degrees
- moved C1 10.4 mm to (144.6, 92.6), turned to 180 degrees
- moved C2 9.64 mm to (143.9, 105.3)
- moved R8 7.16 mm to (144.6, 94.3), turned to 180 degrees
- moved L2 6.42 mm to (161.8, 94.1), turned to 180 degrees
- moved C10 6.37 mm to (161.8, 97.3), turned to 0 degrees
- moved C3 6.35 mm to (160.5, 103.3), turned to 0 degrees
- moved C18 4.99 mm to (168.3, 100.5), turned to 90 degrees
- moved C11 4.50 mm to (161.8, 95.7), turned to 0 degrees
- moved Y1 0.81 mm to (165.4, 100.8), turned to 180 degrees
- turned C17 to 180 degrees
- renumbered C11 to C12, C12 to C13, C13 to C14, C14 to C15, C15 to C16, C16 to C17, C17 to C18, C18 to C19, C19 to C20, C20 to C21, C21 to C22, C5 to C6, C6 to C7, C7 to C8, C8 to C9, SW2 to RESET
Routing:
- net +BATT: track 52.0 -> 29.1 mm, vias 1 -> 2
- net +3.3V: track 311.7 -> 292.6 mm, vias 10 -> 13
- net /AD3: track 45.8 -> 51.8 mm
- net GND: track 0.00 -> 5.83 mm, vias 178 -> 182
- net /OSC_IN: track 13.2 -> 8.30 mm
- net /AD_BATT: track 11.9 -> 15.2 mm, vias 0 -> 2
- net /2.4G_RST: track 26.7 -> 24.0 mm
- net /AD1: track 58.5 -> 56.3 mm
- net /OSC_OUT: track 9.53 -> 11.4 mm
- net +3.3VA: track 5.92 -> 7.09 mm, vias 1 -> 0
- net /BOOT1: track 4.97 -> 6.11 mm, vias 1 -> 0
- net /BOOT0: track 6.49 -> 7.49 mm, vias 1 -> 0
- net /D+: track 10.6 -> 11.6 mm
- net /S5: track 50.8 -> 51.6 mm
- net /CE: track 31.9 -> 31.2 mm
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- added copper zone on B.Cu, net +3.3V
- removed copper zone on In2.Cu, net GND
Other:
- copper layers 4 -> 2
