File: 遥控器/遥控器.kicad_sch (KiCad schematic)
At the start: 36 parts

Commit message: 完成原理图，pcb布局
Parts:
- added C18, C19: 0.1u, Capacitor_SMD:C_0603_1608Metric, symbol Device:C
- added J1, J2: Conn_01x01_Pin, Connector_Wire:SolderWirePad_1x01_SMD_1x2mm, symbol Connector:Conn_01x01_Pin
- added R2: 1k, Resistor_SMD:R_0603_1608Metric, symbol Device:R
- added R4: 150k, Resistor_SMD:R_0603_1608Metric, symbol Device:R
- added R7: 20.5k, Resistor_SMD:R_0603_1608Metric, symbol Device:R
- added SW1: SK12F14G5, Button_Switch_THT:SW-TH_SK12F14G5, symbol Switch:SK12F14G5
- added SW10, SW11, SW12, SW3, SW4, SW5, SW6, SW7, SW8, SW9: SW_Push, Button_Switch_SMD:SW_Push_1P1T_NO_6x6mm_H9.5mm, symbol Switch:SW_Push
- added SW13, SW14: SW_Push, Button_Switch_THT:SW_Tactile_SPST_Angled_PTS645Vx39-2LFS, symbol Switch:SW_Push
- added U2: IPS_1.14_135X240_ST7789_13P顶层, Display:1.14IPS-LCD, symbol Display_Graphic:IPS_1.14_135X240_ST7789_13P顶层
- added U5: 2.4G-UART, RF_Module:2.4G-UART, symbol RF_Module:2.4G-UART
- added U6: W25Q128JVS, Package_SO:SOIC-8_5.23x5.23mm_P1.27mm, symbol Memory_Flash:W25Q128JVS
- added U8: 10k, 摇杆:16x16 360度回中, symbol 摇杆:16x16_360度回中
- added U9: 10k, 摇杆:摇杆16x16一字不回中, symbol 摇杆:16x16不回中
- C1, C10, C11, C12, C13, C14, C15, C16, C17, C2, C20, C21, C3, C4, C5, C6, C7, C8, C9: renamed from C?; footprint (none) -> Capacitor_SMD:C_0603_1608Metric
- D1: renamed from D?; footprint (none) -> Diode_SMD:D_SOD-123
- J3: renamed from J?; footprint (none) -> Connector_USB:USB_C_Receptacle_G-Switch_GT-USB-7010ASV
- L1: renamed from L?; footprint (none) -> Inductor_SMD:L_Chilisin_BMRA00040420
- L2: renamed from L?; footprint (none) -> Inductor_SMD:L_0603_1608Metric
- R1, R10, R3, R5, R6, R8, R9: renamed from R?; footprint (none) -> Resistor_SMD:R_0603_1608Metric
- SW2: renamed from SW?; footprint (none) -> Button_Switch_SMD:SW-SMD_L4.0-W2.9-LS4.8-1
- Y1: renamed from Y?; footprint (none) -> Crystal:Crystal_SMD_3225-4Pin_3.2x2.5mm
- gave numbers to parts that had none: 4
Connections:
- net RX is gone; now on net USART1_RX: U7.6 (TXD)
- net TX is gone; now on net USART1_TX: U7.7 (RXD)
- net +3.3V: now also R5.1, C18.1, C19.2, R2.1, U2.10 (VCC), U2.12 (LEDA), U5.2 (VCC), U6.3 (IO2), U6.7 (IO3), U6.8 (VCC), U8.3 (10k), U8.6 (10k), U9.3 (10k)
- net +3.3VA: now also U3.13 (VDDA)
- net +BATT: now also R4.1, SW1.2
- net BOOT1: now also U3.28 (PB2); no longer U3.26 (PB0)
- net GND: now also Y1.2, Y1.4, C18.2, C19.1, J2.1 (Pin_1), R7.2, SW10.2, SW11.2, SW12.2, SW13.2, SW14.2, SW3.2, SW4.2, SW5.2, SW6.2, SW7.2, SW8.2, SW9.2, U2.11 (LEDK), U2.13 (GND), U2.8 (GND), U5.3 (GND), U5.7 (GND), U6.4 (GND), U8.1 (0), U8.4 (0), U9.1 (0)
- net AD2: now reaches U3.10 (PC2)
- net AD2: now also U8.5 (R)
- net AD3: now reaches U3.11 (PC3)
- net AD3: now also U9.2 (R)
- net 2.4G_RST: now reaches U3.14 (PA0)
- net 2.4G_RST: now also U5.1 (RST)
- net CE: now reaches U3.15 (PA1)
- net CE: now also U5.6 (CE)
- net USART2_TX: now reaches U3.16 (PA2)
- net USART2_TX: now also U5.4 (RX)
- net USART2_RX: now reaches U3.17 (PA3)
- net USART2_RX: now also U5.5 (TX)
- net SPI1_SCL: now reaches U3.21 (PA5)
- net SPI1_SCL: now also R2.2
- net SPI1_SDA: now reaches U3.23 (PA7)
- net SPI1_SDA: now also U2.3 (SDA)
- net RS: now reaches U3.24 (PC4)
- net RS: now also U2.5 (RS)
- net RES: now reaches U3.25 (PC5)
- net RES: now also U2.6 (RES)
- net CS2: now reaches U3.33 (PB12)
- net CS2: now also U6.1 (~{CS})
- net SPI2_SCL: now reaches U3.34 (PB13)
- net SPI2_SCL: now also U2.4 (SCL), U6.6 (CLK)
- net SPI2_MISO: now reaches U3.35 (PB14)
- net SPI2_MISO: now also U6.2 (DO(IO1))
- net SPI2_MOSI: now reaches U3.36 (PB15)
- net SPI2_MOSI: now also U6.5 (DI(IO0))
- net USART1_TX: now reaches U3.42 (PA9)
- net USART1_RX: now reaches U3.43 (PA10)
- net S1: now reaches U3.50 (PA15)
- net S1: now also SW3.1
- net S2: now reaches U3.51 (PC10)
- net S2: now also SW4.1
- net S3: now reaches U3.52 (PC11)
- net S3: now also SW5.1
- net S4: now reaches U3.53 (PC12)
- net S4: now also SW6.1
- net S5: now reaches U3.54 (PD2)
- net S5: now also SW7.1
- net S6: now reaches U3.55 (PB3)
- net S6: now also SW8.1
- net S7: now reaches U3.56 (PB4)
- net S7: now also SW9.1
- net S8: now reaches U3.57 (PB5)
- net S8: now also SW10.1
- net S9: now reaches U3.58 (PB6)
- net S9: now also SW11.1
- net S10: now reaches U3.59 (PB7)
- net S10: now also SW12.1
- net S11: now reaches U3.61 (PB8)
- net S11: now also SW13.1
- net S12: now reaches U3.62 (PB9)
- net S12: now also SW14.1
- net AD_BATT: now reaches U3.8 (PC0)
- net AD_BATT: now also R4.2, R7.1
- net AD1: now reaches U3.9 (PC1)
- net AD1: now also U8.2 (R)
- new net +VDC: J1.1 (Pin_1), SW1.1
- new net CS1: U2.7 (CS), U3.26 (PB0)
- no-connect marks 5 -> 30
Other:
- moved on the sheet: C1, C10, C11, C12, C13, C14, C15, C16, C17, C2, C20, C21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

Commit message: 完成pcb绘制
Parts:
- added J3, J4, J5, J6: Conn_01x01_Pin, Connector_Wire:SolderWirePad_1x01_SMD_1x2mm, symbol Connector:Conn_01x01_Pin
- renumbered J3 to J7
Connections:
- net +3.3V: now also J5.1 (Pin_1)
- net GND: now also J7.S1 (SHIELD), J6.1 (Pin_1)
- net S1: now also U3.45 (PA12); no longer U3.50 (PA15)
- net S10: now also U3.54 (PD2); no longer U3.59 (PB7)
- net S11: now also U3.30 (PB11); no longer U3.61 (PB8)
- net S12: now also U3.29 (PB10); no longer U3.62 (PB9)
- net S2: now also U3.50 (PA15); no longer U3.51 (PC10)
- net S4: now also U3.51 (PC10); no longer U3.53 (PC12)
- net S5: now also U3.58 (PB6); no longer U3.54 (PD2)
- net S6: now also U3.56 (PB4); no longer U3.55 (PB3)
- net S7: now also U3.55 (PB3); no longer U3.56 (PB4)
- net S9: now also U3.59 (PB7); no longer U3.58 (PB6)
- net SPI1_SCL: now also U2.4 (SCL)
- net SPI2_SCL: no longer U2.4 (SCL)
- net SW: now reaches D1.2 (A), L1.1, U1.1 (SW)
- net SWDIO: now reaches U3.46 (PA13)
- net SWDIO: now also J3.1 (Pin_1)
- net SWCLK: now reaches U3.49 (PA14)
- net SWCLK: now also J4.1 (Pin_1)
- no-connect marks 30 -> 27

Commit message: 飞控原理图完成
Parts:
- added C5: 0.1u, Capacitor_SMD:C_0603_1608Metric, symbol Device:C
- renumbered C9 to C10, C10 to C11, C11 to C12, C12 to C13, C13 to C14, C14 to C15, C15 to C16, C16 to C17, C17 to C18, C18 to C19, C19 to C20, C20 to C21, C21 to C22, C5 to C6, C6 to C7, C7 to C8, C8 to C9
Connections:
- net +3.3V: now also C5.1
- net GND: now also C5.2
Changed lines of the file:
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@@
   (junction (at 48.26 24.13) (diameter 0) (color 0 0 0 0)
   )
+  (junction (at 128.27 26.67) (diameter 0) (color 0 0 0 0)
+  )
   (junction (at 181.61 31.75) (diameter 0) (color 0 0 0 0)
   )
@@
   (junction (at 74.93 156.21) (diameter 0) (color 0 0 0 0)
   )
+  (junction (at 128.27 34.29) (diameter 0) (color 0 0 0 0)
+  )
   (junction (at 196.85 77.47) (diameter 0) (color 0 0 0 0)
   )
@@
     (stroke (width 0) (type default))
   )
+  (wire (pts (xy 128.27 26.67) (xy 138.43 26.67))
+    (stroke (width 0) (type default))
+  )
   (wire (pts (xy 50.8 118.11) (xy 52.07 118.11))
     (stroke (width 0) (type default))
   )
+  (wire (pts (xy 128.27 34.29) (xy 138.43 34.29))
+    (stroke (width 0) (type default))
+  )
   (wire (pts (xy 113.03 60.96) (xy 119.38 60.96))
     (stroke (width 0) (type default))
@@
     )
   )
+  (symbol (lib_id "Device:C") (at 138.43 30.48 0) (unit 1)
+    (in_bom yes) (on_board yes) (dnp no) (fields_autoplaced)
+    (property "Reference" "C5" (at 142.24 29.21 0)
+      (effects (font (size 1.27 1.27)) (justify left))
+    )
+    (property "Value" "0.1u" (at 142.24 31.75 0)
+      (effects (font (size 1.27 1.27)) (justify left))
+    )
+    (property "Footprint" "Capacitor_SMD:C_0603_1608Metric" (at 139.3952 34.29 0)
+      (effects (font (size 1.27 1.27)) hide)
+    )
+    (property "Datasheet" "~" (at 138.43 30.48 0)
+      (effects (font (size 1.27 1.27)) hide)
+    )
+    (pin "1")
+    (pin "2")
+    (instances
+      (project "遥控器"
+        (path "/7acf24c7-65ea-488f-bd8e-e40e18ad27a1"
+          (reference "C5") (unit 1)
+        )
+      )
+    )
+  )
   (symbol (lib_id "power:+BATT") (at 207.01 24.13 0) (unit 1)
     (in_bom yes) (on_board yes) (dnp no) (fields_autoplaced)
@@
   (symbol (lib_id "Device:C") (at 187.96 44.45 0) (unit 1)
     (in_bom yes) (on_board yes) (dnp no)
-    (property "Reference" "C8" (at 190.5 43.18 0)
+    (property "Reference" "C9" (at 190.5 43.18 0)
       (effects (font (size 1.27 1.27)) (justify left))
     )
@@
       (project "遥控器"
         (path "/7acf24c7-65ea-488f-bd8e-e40e18ad27a1"
-          (reference "C8") (unit 1)
+          (reference "C9") (unit 1)
         )
       )
@@
   (symbol (lib_id "Device:C") (at 113.03 154.94 270) (unit 1)
     (in_bom yes) (on_board yes) (dnp no) (fields_autoplaced)
-    (property "Reference" "C20" (at 113.03 147.32 90)
+    (property "Reference" "C21" (at 113.03 147.32 90)
       (effects (font (size 1.27 1.27)))
     )
@@
       (project "遥控器"
         (path "/7acf24c7-65ea-488f-bd8e-e40e18ad27a1"
-          (reference "C20") (unit 1)
+          (reference "C21") (unit 1)
         )
       )
@@
   (symbol (lib_id "Device:C") (at 99.06 106.68 180) (unit 1)
     (in_bom yes) (on_board yes) (dnp no) (fields_autoplaced)
-    (property "Reference" "C16" (at 91.44 106.68 90)
+    (property "Reference" "C17" (at 91.44 106.68 90)
       (effects (font (size 1.27 1.27)))
     )
@@
       (project "遥控器"
         (path "/7acf24c7-65ea-488f-bd8e-e40e18ad27a1"
-          (reference "C16") (unit 1)
+          (reference "C17") (unit 1)
         )
       )
@@
   (symbol (lib_id "Device:C") (at 124.46 106.68 180) (unit 1)
     (in_bom yes) (on_board yes) (dnp no) (fields_autoplaced)
-    (property "Reference" "C17" (at 116.84 106.68 90)
+    (property "Reference" "C18" (at 116.84 106.68 90)
       (effects (font (size 1.27 1.27)))
     )
@@
       (project "遥控器"
         (path "/7acf24c7-65ea-488f-bd8e-e40e18ad27a1"
-          (reference "C17") (unit 1)
+          (reference "C18") (unit 1)
         )
       )
@@
   (symbol (lib_id "Device:C") (at 240.03 39.37 0) (unit 1)
     (in_bom yes) (on_board yes) (dnp no) (fields_autoplaced)
-    (property "Reference" "C6" (at 243.84 38.1 0)
+    (property "Reference" "C7" (at 243.84 38.1 0)
       (effects (font (size 1.27 1.27)) (justify left))
     )
@@
       (project "遥控器"
         (path "/7acf24c7-65ea-488f-bd8e-e40e18ad27a1"
-          (reference "C6") (unit 1)
+          (reference "C7") (unit 1)
         )
       )
@@
   (symbol (lib_id "Device:C") (at 213.36 133.35 90) (unit 1)
     (in_bom yes) (on_board yes) (dnp no) (fields_autoplaced)
-    (property "Reference" "C18" (at 213.36 125.73 90)
+    (property "Reference" "C19" (at 213.36 125.73 90)
       (effects (font (size 1.27 1.27)))
     )
@@
       (project "遥控器"
         (path "/7acf24c7-65ea-488f-bd8e-e40e18ad27a1"
-          (reference "C18") (unit 1)
+          (reference "C19") (unit 1)
         )
       )
@@
   (symbol (lib_id "Device:C") (at 284.48 146.05 180) (unit 1)
     (in_bom yes) (on_board yes) (dnp no) (fields_autoplaced)
-    (property "Reference" "C19" (at 288.29 144.78 0)
+    (property "Reference" "C20" (at 288.29 144.78 0)
       (effects (font (size 1.27 1.27)) (justify right))
     )
@@
       (project "遥控器"
         (path "/7acf24c7-65ea-488f-bd8e-e40e18ad27a1"
-          (reference "C19") (unit 1)
+          (reference "C20") (unit 1)
         )
       )
@@
   (symbol (lib_id "Device:C") (at 234.95 83.82 0) (unit 1)
     (in_bom yes) (on_board yes) (dnp no) (fields_autoplaced)
-    (property "Reference" "C15" (at 238.76 82.55 0)
+    (property "Reference" "C16" (at 238.76 82.55 0)
       (effects (font (size 1.27 1.27)) (justify left))
     )
@@
       (project "遥控器"
         (path "/7acf24c7-65ea-488f-bd8e-e40e18ad27a1"
-          (reference "C15") (unit 1)
+          (reference "C16") (unit 1)
         )
       )
@@
   (symbol (lib_id "Device:C") (at 196.85 83.82 0) (unit 1)
     (in_bom yes) (on_board yes) (dnp no) (fields_autoplaced)
-    (property "Reference" "C13" (at 200.66 82.55 0)
+    (property "Reference" "C14" (at 200.66 82.55 0)
       (effects (font (size 1.27 1.27)) (justify left))
     )
@@
       (project "遥控器"
         (path "/7acf24c7-65ea-488f-bd8e-e40e18ad27a1"
-          (reference "C13") (unit 1)
+          (reference "C14") (unit 1)
         )
       )
@@
   (symbol (lib_id "Device:C") (at 222.25 83.82 0) (unit 1)
     (in_bom yes) (on_board yes) (dnp no) (fields_autoplaced)
-    (property "Reference" "C14" (at 226.06 82.55 0)
+    (property "Reference" "C15" (at 226.06 82.55 0)
       (effects (font (size 1.27 1.27)) (justify left))
     )
@@
       (project "遥控器"
         (path "/7acf24c7-65ea-488f-bd8e-e40e18ad27a1"
-          (reference "C14") (unit 1)
+          (reference "C15") (unit 1)
         )
       )
@@
   (symbol (lib_id "Device:C") (at 123.19 158.75 180) (unit 1)
     (in_bom yes) (on_board yes) (dnp no) (fields_autoplaced)
-    (property "Reference" "C21" (at 127 157.48 0)
+    (property "Reference" "C22" (at 127 157.48 0)
       (effects (font (size 1.27 1.27)) (justify right))
     )
@@
       (project "遥控器"
         (path "/7acf24c7-65ea-488f-bd8e-e40e18ad27a1"
-          (reference "C21") (unit 1)
+          (reference "C22") (unit 1)
         )
       )
@@
   (symbol (lib_id "Device:C") (at 186.69 83.82 0) (unit 1)
     (in_bom yes) (on_board yes) (dnp no) (fields_autoplaced)
-    (property "Reference" "C12" (at 190.5 82.55 0)
+    (property "Reference" "C13" (at 190.5 82.55 0)
       (effects (font (size 1.27 1.27)) (justify left))
     )
@@
       (project "遥控器"
         (path "/7acf24c7-65ea-488f-bd8e-e40e18ad27a1"
-          (reference "C12") (unit 1)
+          (reference "C13") (unit 1)
         )
       )
@@
   (symbol (lib_id "Device:C") (at 95.25 82.55 0) (unit 1)
     (in_bom yes) (on_board yes) (dnp no) (fields_autoplaced)
-    (property "Reference" "C11" (at 99.06 81.28 0)
+    (property "Reference" "C12" (at 99.06 81.28 0)
       (effects (font (size 1.27 1.27)) (justify left))
     )
@@
       (project "遥控器"
         (path "/7acf24c7-65ea-488f-bd8e-e40e18ad27a1"
-          (reference "C11") (unit 1)
+          (reference "C12") (unit 1)
         )
       )
@@
   (symbol (lib_id "Device:C") (at 106.68 57.15 0) (unit 1)
     (in_bom yes) (on_board yes) (dnp no) (fields_autoplaced)
-    (property "Reference" "C9" (at 110.49 55.88 0)
+    (property "Reference" "C10" (at 110.49 55.88 0)
       (effects (font (size 1.27 1.27)) (justify left))
     )
@@
       (project "遥控器"
         (path "/7acf24c7-65ea-488f-bd8e-e40e18ad27a1"
-          (reference "C9") (unit 1)
+          (reference "C10") (unit 1)
         )
       )
@@
   (symbol (lib_id "Device:C") (at 175.26 44.45 0) (unit 1)
     (in_bom yes) (on_board yes) (dnp no) (fields_autoplaced)
-    (property "Reference" "C7" (at 179.07 43.18 0)
+    (property "Reference" "C8" (at 179.07 43.18 0)
       (effects (font (size 1.27 1.27)) (justify left))
     )
@@
       (project "遥控器"
         (path "/7acf24c7-65ea-488f-bd8e-e40e18ad27a1"
-          (reference "C7") (unit 1)
+          (reference "C8") (unit 1)
         )
       )
@@
   (symbol (lib_id "Device:C") (at 229.87 39.37 0) (unit 1)
     (in_bom yes) (on_board yes) (dnp no) (fields_autoplaced)
-    (property "Reference" "C5" (at 233.68 38.1 0)
+    (property "Reference" "C6" (at 233.68 38.1 0)
       (effects (font (size 1.27 1.27)) (justify left))
     )
@@
       (project "遥控器"
         (path "/7acf24c7-65ea-488f-bd8e-e40e18ad27a1"
-          (reference "C5") (unit 1)
+          (reference "C6") (unit 1)
         )
       )
@@
   (symbol (lib_id "Device:C") (at 119.38 57.15 0) (unit 1)
     (in_bom yes) (on_board yes) (dnp no) (fields_autoplaced)
-    (property "Reference" "C10" (at 123.19 55.88 0)
+    (property "Reference" "C11" (at 123.19 55.88 0)
       (effects (font (size 1.27 1.27)) (justify left))
     )
@@
       (project "遥控器"
         (path "/7acf24c7-65ea-488f-bd8e-e40e18ad27a1"
-          (reference "C10") (unit 1)
+          (reference "C11") (unit 1)
         )
       )
