File: 飞控/飞控.kicad_sch (KiCad schematic)
At the start: 44 parts

Commit message: 原理图批注
Parts:
- added J? (x4): Conn_01x02_Pin, symbol Connector:Conn_01x02_Pin
- added Q? (x4): AO3400A, Package_TO_SOT_SMD:SOT-23, symbol Transistor_FET:AO3400A
- added R? (x4): 10, symbol Device:R
- added R? (x4): 10k, symbol Device:R
Connections:
- net +BATT: now also J?.2 (Pin_2), J?.2 (Pin_2), J?.2 (Pin_2), J?.2 (Pin_2)
- net GND: now also Q?.2 (S), Q?.2 (S), Q?.2 (S), Q?.2 (S), R?.2, R?.2, R?.2, R?.2
- net PWM1: now also R?.1
- net PWM2: now also R?.1
- net PWM3: now also R?.1
- net PWM4: now also R?.1
- new net: Q?.1 (G), R?.1, R?.2 (x4)
- new net: J?.1 (Pin_1), Q?.3 (D) (x4)
Other:
- moved on the sheet: C?, D?, L?, R?, SW?, U?, Y?

Commit message: 批注原理图
Parts:
- gave numbers to parts that had none: 60

Commit message: 飞控原理图完成
Parts:
- removed D2: LED, symbol Device:LED
- removed D4: D, symbol Device:D
- removed J1, J2, J3, J4: Conn_01x02_Pin, symbol Connector:Conn_01x02_Pin
- removed R16, R17: 10, symbol Device:R
- removed R18, R20: 10k, symbol Device:R
- removed R19: 20.5k, symbol Device:R
- removed U1: GD32F103TBU6, kicad_lceda:QFN-36_L6.0-W6.0-P0.50-BL-EP3.9, symbol GigaDevice:GD32F103TBU6
- removed U2: MPU-6050, Sensor_Motion:InvenSense_QFN-24_4x4mm_P0.5mm, symbol Sensor_Motion:MPU-6050
- removed U3: ME6206A33M3G, Package_TO_SOT_SMD:SOT-23, symbol Regulator_Linear:ME6206A33M3G
- removed U4: 2.4G-UART, RF_Module:2.4G-UART, symbol RF_Module:2.4G-UART
- removed U5: SX1308, Package_TO_SOT_SMD:SOT-23-6, symbol Converter_DCDC:SX1308
- added C21, C22, C23: 0.1u, Capacitor_SMD:C_0603_1608Metric, symbol Device:C
- added D2, D5, D6, D7, D8: 1N5819, Diode_SMD:D_SOD-123, symbol Device:D
- added D4: LED, LED_SMD:LED_0603_1608Metric, symbol Device:LED
- added H1, H2, H3, H4: MountingHole_Pad, MountingHole:hole_2x3mm, symbol Mechanical:MountingHole_Pad
- added J1: BATT_IN, symbol Connector:Conn_01x02_Socket
- added J2: Conn_01x06_Pin, Connector_Wire:WirePad_1x06_1.5mm, symbol Connector:Conn_01x06_Pin
- added J3: Conn_01x03, Connector_PinHeader_2.54mm:PinHeader_1x03_P2.54mm_Vertical, symbol Connector_Generic:Conn_01x03
- added J4: M1_OUT, Connector_Wire:WIrePad_1x02_2mm, symbol Connector:Conn_01x02_Socket
- added J5: M2_OUT, Connector_Wire:WIrePad_1x02_2mm, symbol Connector:Conn_01x02_Socket
- added J6: M3_OUT, Connector_Wire:WIrePad_1x02_2mm, symbol Connector:Conn_01x02_Socket
- added J7: M4_OUT, Connector_Wire:WIrePad_1x02_2mm, symbol Connector:Conn_01x02_Socket
- added U1: SX1308, Package_TO_SOT_SMD:SOT-23-6, symbol Converter_DCDC:SX1308
- added U2: 2.4G-UART, RF_Module:2.4G-UART, symbol RF_Module:2.4G-UART
- added U3: BMP280, Package_LGA:Bosch_LGA-8_2x2.5mm_P0.65mm_ClockwisePinNumbering, symbol Sensor_Pressure:BMP280
- added U4: ME6206A33M3G, Package_TO_SOT_SMD:SOT-23, symbol Regulator_Linear:ME6206A33M3G
- added U5: SS12D06弯针, Button_Switch_THT:SW-TH_3P-SS12D06-1, symbol Switch:SS12D06弯针
- added U6: W25Q32JVSS, Package_SO:SOIC-8_5.23x5.23mm_P1.27mm, symbol Memory_Flash:W25Q32JVSS
- added U7: MPU-6050, Package_DFN_QFN:QFN-24-1EP_4x4mm_P0.5mm_EP2.6x2.6mm, symbol Sensor_Motion:MPU-6050
- added U8: GD32F103TBU6, Package_DFN_QFN:QFN-36-1EP_6x6mm_P0.5mm_EP3.7x3.7mm, symbol GigaDevice:GD32F103TBU6
- C1: value 20p -> 0.1u; footprint (none) -> Capacitor_SMD:C_0603_1608Metric
- C10, C14, C15, C18, C2, C4, C6, C7, C8, C9: footprint (none) -> Capacitor_SMD:C_0603_1608Metric
- C11, C13, C16, C17: value 22u -> 0.1u; footprint (none) -> Capacitor_SMD:C_0603_1608Metric
- C12: value 0.1u -> 4.7u; footprint (none) -> Capacitor_SMD:C_0603_1608Metric
- C19: value 0.1u -> 22p; footprint (none) -> Capacitor_SMD:C_0603_1608Metric
- C20: value 22u -> 22p; footprint (none) -> Capacitor_SMD:C_0603_1608Metric
- C3: value 20p -> 22u; footprint (none) -> Capacitor_SMD:C_0603_1608Metric
- C5: value 0.1u -> 22u; footprint (none) -> Capacitor_SMD:C_0603_1608Metric
- D1, D3: footprint (none) -> LED_SMD:LED_0603_1608Metric
- L1: value L -> 4.7u; footprint (none) -> Inductor_SMD:IND-SMD_L4.0-W4.0_0.47UH04209.5A
- R1, R13, R14, R4, R8: footprint (none) -> Resistor_SMD:R_0603_1608Metric
- R10: value 100k -> 10k; footprint (none) -> Resistor_SMD:R_0603_1608Metric
- R11, R12: value 10 -> 10k; footprint (none) -> Resistor_SMD:R_0603_1608Metric
- R15, R5: value 150k -> 10k; footprint (none) -> Resistor_SMD:R_0603_1608Metric
- R2: value 4.7k -> 10k; footprint (none) -> Resistor_SMD:R_0603_1608Metric
- R3: value 4.7k -> 150k; footprint (none) -> Resistor_SMD:R_0603_1608Metric
- R6: value 1k -> 20.5k; footprint (none) -> Resistor_SMD:R_0603_1608Metric
- R7: value 1k -> 10k; footprint (none) -> Resistor_SMD:R_0603_1608Metric
- R9: value 10k -> 1k; footprint (none) -> Resistor_SMD:R_0603_1608Metric
- SW1: value SW_Push -> RST; footprint (none) -> Button_Switch_SMD:SW-SMD_L4.0-W2.9-LS4.8-1
- Y1: footprint (none) -> Crystal:Crystal_SMD_3225-4Pin_3.2x2.5mm
Connections:
- net AD0 is gone; now on an unnamed net: R4.2
- net LED3 is gone; now on net LED2: D3.1 (K)
- net SCL is gone; now on net +BATT: R2.1
- net SDA is gone; now on net +5V: R3.1
- net +3.3V: now also C1.1, C10.1, C11.1, C12.1, C13.1, C14.1, C15.1, C16.1, C17.1, C18.1, C2.1, C9.1, R1.1, R13.2, R4.1, R7.1, R8.1, R9.1, J2.1 (Pin_1), U2.2 (VCC), U3.6 (VDDIO), U3.8 (VDD), U4.2 (OUT), U6.3 (IO2), U6.7 (IO3), U6.8 (VCC), U7.13 (VDD), U7.8 (VLOGIC), U8.1 (VDD_3), U8.19 (VDD_1), U8.27 (VDD_2), U8.6 (VDDA); no longer C10.2, C15.2, C2.2, C7.2, C8.2, C9.2, R2.2, R3.2, R6.2, R7.2, R8.2, R9.2
- net +5V: now also C3.1, C4.1, C7.1, C8.1, D2.1 (K), J3.1 (Pin_1), U4.3 (VIN); no longer C11.2, C12.2, C19.2, C20.2, R15.2
- net +BATT: now also C5.1, C6.1, L1.2, D5.1 (K), D6.1 (K), D7.1 (K), D8.1 (K), J4.1 (Pin_1), J5.1 (Pin_1), J6.1 (Pin_1), J7.1 (Pin_1), U1.4 (EN), U1.5 (IN), U5.3; no longer C16.2, C17.2, C18.2, L1.1, R5.2
- net FB: now also R3.2, R6.1, U1.3 (FB); no longer R15.1
- net GND: now also C1.2, C10.2, C11.2, C12.2, C13.2, C14.2, C15.2, C16.2, C17.2, C18.2, C2.2, C3.2, C4.2, C5.2, C6.2, C7.2, C8.2, C9.2, R10.2, R11.2, R12.2, R15.2, R5.2, R6.2, Y1.2, Y1.4, C21.1, C22.1, C23.2, D4.1 (K), H1.1, H2.1, H3.1, H4.1, J1.2 (Pin_2), J2.6 (Pin_6), J3.3 (Pin_3), U1.2 (GND), U2.3 (GND), U2.7 (GND), U3.1 (GND), U3.7 (GND), U4.1 (GND), U6.4 (GND), U7.1 (CLKIN), U7.11 (FSYNC), U7.18 (GND), U7.9 (AD0), U8.18 (VSS_1), U8.26 (VSS_2), U8.36 (VSS_3), U8.37 (EP), U8.5 (VSSA); no longer C10.1, C11.1, C12.1, C13.1, C14.1, C15.1, C16.1, C17.1, C18.1, C2.1, C6.1, C7.1, C8.1, C9.1, R1.2, R10.1, R13.2, R4.1
- net LED1: now also U8.24 (PA12)
- net LED2: now also U8.23 (PA11)
- net NRST: now also R13.1, C23.1, U8.4 (NRST); no longer C6.2, R9.1
- net PWM1: now also Q2.1 (G), R11.1, U8.31 (PB4); no longer R12.1
- net PWM2: now also Q1.1 (G), R10.1, U8.32 (PB5); no longer R11.1
- net PWM3: now also Q3.1 (G), R14.1, U8.16 (PB1)
- net PWM4: now also Q4.1 (G), R15.1, U8.15 (PB0)
- net M3: now reaches Q3.3 (D)
- net M3: now also D7.2 (A), J6.2 (Pin_2)
- net OSC_OUT: now reaches Y1.1
- net OSC_OUT: now also C20.2, U8.3 (OSC_OUT/PD1); no longer C3.2
- net M4: now reaches Q4.3 (D)
- net M4: now also D8.2 (A), J7.2 (Pin_2)
- net at D3.2 (A): no longer R8.1
- net M1: now reaches Q1.3 (D)
- net M1: now also D5.2 (A), J4.2 (Pin_2)
- net M2: now reaches Q2.3 (D)
- net M2: now also D6.2 (A), J5.2 (Pin_2)
- net OSC_IN: now reaches Y1.3
- net OSC_IN: now also C19.2, U8.2 (OSC_IN/PD0); no longer C1.2
- net at D1.2 (A): now also R1.2; no longer R6.1
- net ADC renamed BAT_ADC
- net BAT_ADC: now also R2.2, U8.7 (PA0-WKUP); no longer R10.2
- new net: D2.2 (A), L1.1, U1.1 (SW)
- new net: D4.2 (A), R7.2
- new net: R12.1, U8.35 (BOOT0)
- new net: C21.2, U7.10 (REGOUT)
- new net: C22.2, U7.20 (CPOUT)
- new net 6050_INT: U7.12 (INT), U8.30 (PB3)
- new net 6050_SCL: R8.2, U7.23 (SCL), U8.33 (PB6)
- new net 6050_SDA: R9.2, U7.24 (SDA), U8.34 (PB7)
- new net BMP280_CS: U3.2 (CSB), U8.17 (PB2)
- new net SPI_CS: U6.1 (~{CS}), U8.11 (PA4)
- new net SPI_MISO: U3.5 (SDO), U6.2 (DO(IO1)), U8.13 (PA6)
- new net SPI_MOSI: U3.3 (SDI), U6.5 (DI(IO0)), U8.14 (PA7)
- new net SPI_SCK: U3.4 (SCK), U6.6 (CLK), U8.12 (PA5)
- new net SWCLK: J2.2 (Pin_2), U8.28 (PA14)
- new net SWDIO: J2.3 (Pin_3), U8.25 (PA13)
- new net U1_RX: J2.4 (Pin_4), J3.2 (Pin_2), U8.22 (PA10)
- new net U1_TX: J2.5 (Pin_5), U8.21 (PA9)
- new net U2_RX: U2.5 (TX), U8.10 (PA3)
- new net U2_TX: U2.4 (RX), U8.9 (PA2)
- new net UART_RST: U2.1 (RST), U8.8 (PA1)
- new net VIN: J1.1 (Pin_1), U5.2
- no-connect marks 2 -> 7
Other:
- note added: "8M FLASH"
- note added: "MPU-6050"
- note added: "指示灯"
- note added: "摄像头"
- note added: "无线通信"
- note added: "最小系统"
- note added: "气压计"
- note added: "电压监测"
- note added: "电机输出"
- note added: "电源管理"
- note added: "电源输入"
- note added: "调试接口"

Commit message: 飞控pcb布局
Connections:
- net SW: now reaches D2.2 (A), L1.1, U1.1 (SW)
Changed lines of the file:
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@@
     (effects (font (size 1.27 1.27)) (justify right bottom))
+  )
+  (label "SW" (at 73.66 55.88 0) (fields_autoplaced)
+    (effects (font (size 1.27 1.27)) (justify left bottom))
   )
   (label "PWM4" (at 220.98 246.38 180) (fields_autoplaced)

Commit message: 飞控修改
Parts:
- removed J1: BATT_IN, symbol Connector:Conn_01x02_Socket
- removed J2: Conn_01x06_Pin, Connector_Wire:WirePad_1x06_1.5mm, symbol Connector:Conn_01x06_Pin
- removed J3: Conn_01x03, Connector_PinHeader_2.54mm:PinHeader_1x03_P2.54mm_Vertical, symbol Connector_Generic:Conn_01x03
- removed J4: M1_OUT, Connector_Wire:WIrePad_1x02_2mm, symbol Connector:Conn_01x02_Socket
- removed J5: M2_OUT, Connector_Wire:WIrePad_1x02_2mm, symbol Connector:Conn_01x02_Socket
- removed J6: M3_OUT, Connector_Wire:WIrePad_1x02_2mm, symbol Connector:Conn_01x02_Socket
- removed J7: M4_OUT, Connector_Wire:WIrePad_1x02_2mm, symbol Connector:Conn_01x02_Socket
- removed U5: SS12D06弯针, Button_Switch_THT:SW-TH_3P-SS12D06-1, symbol Switch:SS12D06弯针
- added CN1: ZH1.5-2P-WT, my_conn:CONN-SMD_ZH1.5-2P-WT, symbol my_conn:ZH1.5-2P-WT
- added J1, J10, J2, J3, J8, J9: Conn_01x01_Pin, TestPoint:TestPoint_Pad_D1.0mm, symbol Connector:Conn_01x01_Pin
- added J11, J12, J13, J14, J4, J5, J6, J7: Conn_01x01_Pin, Connector_Wire:SolderWirePad_1x01_SMD_1x2mm, symbol Connector:Conn_01x01_Pin
- added SW2: MST22D18G2_125, my_switch:SW-SMD_MST22D18G2, symbol my_switch:MST22D18G2_125
- added U9: ZX-ZH1.5-3PWT, my_conn:CONN-SMD_3P-P1.50_ZX-ZH1.5-3PWT, symbol my_conn:ZX-ZH1.5-3PWT
- L1: footprint Inductor_SMD:IND-SMD_L4.0-W4.0_0.47UH04209.5A -> Inductor_SMD:IND-SMD_L4.9-W4.4_MAPM0420F
- U2: footprint RF_Module:2.4G-UART -> my_module:2.4G-UART
Connections:
- net +3.3V: now also J1.1 (Pin_1)
- net +5V: now also U9.1
- net +BATT: now also J12.1 (Pin_1), J4.1 (Pin_1), J5.1 (Pin_1), J6.1 (Pin_1), SW2.1, SW2.4
- net 6050_SCL: now also U8.34 (PB7); no longer U8.33 (PB6)
- net 6050_SDA: now also U8.33 (PB6); no longer U8.34 (PB7)
- net GND: now also CN1.2, J10.1 (Pin_1), U9.3
- net M1: now also J11.1 (Pin_1)
- net M2: now also J13.1 (Pin_1)
- net M3: now also J14.1 (Pin_1)
- net M4: now also J7.1 (Pin_1)
- net SWCLK: now also J2.1 (Pin_1)
- net SWDIO: now also J3.1 (Pin_1)
- net U1_RX: now also J8.1 (Pin_1), U9.2
- net U1_TX: now also J9.1 (Pin_1)
- net VIN: now also CN1.1, SW2.2, SW2.5
- no-connect marks 7 -> 10
